File: pcb/microkvs-stress-test.kicad_sch (KiCad schematic)
At the start: 66 parts, among them J1 BARREL_JACK, J2 PMOD_HOST, J3 XILINX_JTAG, J4 XILINX_JTAG, U1 STM32L431-QFN32, U2 STM32L431-QFN32, U3 W25Q128JV, U4 NCP45521IMNTWG-H

Commit message: Finished initial microkvs-stress-test board design
Parts:
- added M1, M2, M3, M4: SCREWHOLE, azonenberg_pcb:MECHANICAL_CLEARANCEHOLE_4_40, symbol conn:CONN_01X01
- added M5: LOGO_OSHW, w_logo:Logo_silk_OSHW_6x6mm, symbol special-azonenberg:MECHANICAL
- added M6: LONGTHING, azonenberg_pcb:LONGTHING-1200DPI, symbol special-azonenberg:MECHANICAL
- added M7: LOGO_WEEE, w_logo:Logo_silk_WEEE_3.4x5mm, symbol special-azonenberg:MECHANICAL
- C10, C11, C3, C5, C6, C7, C9: footprint (none) -> azonenberg_pcb:EIA_0402_CAP_NOSILK
- C2, C4, C8: footprint (none) -> azonenberg_pcb:EIA_0603_CAP_NOSILK
- D1, D2, D3, D4, D5, D6, D7, D8, D9: footprint (none) -> azonenberg_pcb:EIA_0603_LED
- J1: footprint (none) -> azonenberg_pcb:CONN_CUI_PJ-058BH_HIPWR_BARREL_NOSLOT
- J2: footprint (none) -> azonenberg_pcb:CONN_HEADER_2.54MM_2x6_RA_PMOD_HOST
- J3, J4: footprint (none) -> azonenberg_pcb:XILINX_JTAG_PTH_MOLEX_0878311420
- R1, R10, R12, R13, R14, R15, R16, R17, R18, R19, R2, R20, R22, R23, R24, R27, R28, R29, R3, R30, R31, R32, R33, R34, R4, R5, R6, R7, R8, R9: footprint (none) -> azonenberg_pcb:EIA_0402_RES_NOSILK
- TP2: footprint (none) -> azonenberg_pcb:CONN_HEADER_2.54MM_1x8
- U1, U2: footprint (none) -> azonenberg_pcb:QFN_32_0.5MM_5x5MM
- U3: footprint (none) -> azonenberg_pcb:DFN_8_1.27MM_6x5MM
- U4: footprint (none) -> azonenberg_pcb:DFN_8_0.5MM_2x2MM
Connections:
- net CROSS_FAILDET: now also TP2.7 (P7), U1.18 (PA8); no longer TP2.1 (P1), U1.6 (PA0)
- net CROSS_SPI_MOSI: now also TP2.5 (P5); no longer TP2.7 (P7)
- net CROSS_SPI_SCK: now also TP2.3 (P3); no longer TP2.5 (P5)
- net CTRL_QSPI_DQ1: now also J2.9 (D6); no longer J2.4 (D3)
- net CTRL_QSPI_DQ2: now also J2.4 (D3); no longer J2.7 (D4)
- net CTRL_QSPI_DQ3: now also J2.10 (D7); no longer J2.8 (D5)
- net CTRL_QSPI_SCK: now also J2.8 (D5); no longer J2.1 (D0)
- net DUT_PWREN: now also TP2.1 (P1), U1.6 (PA0); no longer TP2.3 (P3), U1.18 (PA8)
- net DUT_GPIO1: now reaches U2.2 (PC14)
- net DUT_GPIO1: now also J2.7 (D4)
- net DUT_GPIO0: now reaches U2.18 (PA8)
- net DUT_GPIO0: now also J2.1 (D0)
Other:
- moved on the sheet: TP2
